File: pcb/travel-router.kicad_pcb (KiCad board)
At the start: 4 copper layers, 100 x 100 mm, 52 parts, among them J1 USB_C_Receptacle_USB2.0_14P, J2 Conn_02x05_Odd_Even, J5 HDMI_A, J6 JST_SHBM048-SRSS-TB, J8 USB_A_Stacked, SW1 SW_Push, U1 RT9742SNGV, U2 AP2553W6, U3 MagJack-A70-112-331N126, U4 TPD4EUSB30, U5 TPD4EUSB30, U6 RTL8111H-CG, U7 MagJack-A70-112-331N126, U8 TPD4EUSB30, U9 TPD4EUSB30, Y1 XL2EL89COI-111YLC-25M

Commit message: thing
Parts:
- removed J5: HDMI_A, Connector_Video:HDMI_A_Molex_208658-1001_Horizontal
- added U10: TPD4EUSB30, Package_SON:USON-10_2.5x1.0mm_P0.5mm, F.Cu at (109.2, 73.0)
- added U11: TPD2E2U06DCK, Package_TO_SOT_SMD:SOT-323_SC-70, F.Cu at (150.0, 135.6)
- added U12: 476591100, easyeda2kicad:HDMI-SMD_19P-P0.50_0476591102, F.Cu at (112.7, 63.8)
- moved C3 10.1 mm to (107.8, 65.2), turned to 180 degrees
- moved U1 9.86 mm to (107.2, 67.5), turned to 180 degrees
- moved C4 9.12 mm to (108.7, 70.0), turned to -90 degrees
- moved R3 0.25 mm to (183.8, 61.5)
- moved R2 0.15 mm to (183.9, 59.5)
Connections:
- J8 pad 2: /CM5_HighSpeed/USB3-2-D+ -> /CM5_HighSpeed/USB3-1-D-
- J8 pad 3: /CM5_HighSpeed/USB3-2-D- -> /CM5_HighSpeed/USB3-1-D+
- J8 pad 6: /CM5_HighSpeed/USB3-1-D- -> /CM5_HighSpeed/USB3-2-D-
- J8 pad 7: /CM5_HighSpeed/USB3-1-D+ -> /CM5_HighSpeed/USB3-2-D+
Routing:
- net /VBUS: track 131.6 -> 18.8 mm, vias 5 -> 6
- net GND: track 158.4 -> 192.5 mm, vias 150 -> 127
- net /CM5_HighSpeed/HDMI0_TX2+: track 22.9 -> 5.41 mm
- net /CM5_HighSpeed/HDMI0_TX2-: track 22.9 -> 5.41 mm
- net /CM5_HighSpeed/HDMI0_TX1+: track 20.8 -> 5.54 mm
- net /CM5_HighSpeed/HDMI0_TX1-: track 20.8 -> 5.56 mm
- net /CM5_HighSpeed/HDMI0_TX0+: track 18.9 -> 5.66 mm
- net /CM5_HighSpeed/HDMI0_TX0-: track 18.9 -> 5.66 mm
- net /CM5_HighSpeed/HDMI0_CLK+: track 17.1 -> 5.79 mm
- net /CM5_HighSpeed/HDMI0_CLK-: track 17.1 -> 5.79 mm
- net /CM5_HighSpeed/HDMI0_SCL: track 14.6 -> 5.57 mm
- net /CM5_HighSpeed/HDMI0_SDA: track 17.5 -> 8.86 mm
- net /CM5_HighSpeed/HDMI0_CEC: track 23.4 -> 15.8 mm
- net /CM5_HighSpeed/USB3-2-D+: track 19.1 -> 23.5 mm, vias 2 -> 0
- net /CM5_HighSpeed/HDMI0_HOTPLUG: track 22.7 -> 19.1 mm
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