File: pcb/travel-router.kicad_pcb (KiCad board)
At the start: 4 copper layers, 100 x 100 mm, 54 parts, among them J1 USB_C_Receptacle_USB2.0_14P, J2 Conn_02x05_Odd_Even, J6 JST_SHBM048-SRSS-TB, J8 USB_A_Stacked, SW1 SW_Push, U1 RT9742SNGV, U10 TPD4EUSB30, U11 TPD2E2U06DCK, U12 476591100, U2 AP2553W6, U3 MagJack-A70-112-331N126, U4 TPD4EUSB30, U5 TPD4EUSB30, U6 RTL8111H-CG, U7 MagJack-A70-112-331N126, U8 TPD4EUSB30, U9 TPD4EUSB30, Y1 XL2EL89COI-111YLC-25M

Commit message: Create README.md
Parts:
- R2, R3: value 1k -> 1K
Changed lines of the file:
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@@
 			)
 		)
-		(property "Value" "1k"
+		(property "Value" "1K"
 			(at 0 1.17 0)
 			(layer "F.Fab")
@@
 			)
 		)
-		(property "Value" "1k"
+		(property "Value" "1K"
 			(at 0 1.17 0)
 			(layer "F.Fab")

Commit message: pcb stuff
Parts:
- moved H4 0.57 mm to (183.3, 142.9)
- moved H3 0.46 mm to (93.3, 142.9)
- moved H1 0.34 mm to (93.3, 52.9)
- moved H2 0.16 mm to (183.3, 52.9)
Changed lines of the file:
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@@
 	(footprint "MountingHole:MountingHole_3.2mm_M3"
 		(layer "F.Cu")
-		(at 183.7 143.3)
+		(at 183.3 142.9)
 		(descr "Mounting Hole 3.2mm, M3, no annular, generated by kicad-footprint-generator mountinghole.py")
 		(tags "mountinghole M3")
@@
 		)
 		(embedded_fonts no)
-		(model "${KICAD10_3DMODEL_DIR}/Connector_USB.3dshapes/USB_C_Receptacle_HRO_TYPE-C-31-M-12.step"
-			(offset
-				(xyz 0 0 0)
-			)
-			(scale
-				(xyz 1 1 1)
-			)
-			(rotate
-				(xyz 0 0 0)
-			)
-		)
 		(model "${KICAD10_3DMODEL_DIR}/Connector_USB.3dshapes/USB_C_Receptacle_GCT_USB4105-xx-A_16P_TopMnt_Horizontal.step"
 			(offset
@@
 	(footprint "MountingHole:MountingHole_3.2mm_M3"
 		(layer "F.Cu")
-		(at 183.25 52.75)
+		(at 183.3 52.9)
 		(descr "Mounting Hole 3.2mm, M3, no annular, generated by kicad-footprint-generator mountinghole.py")
 		(tags "mountinghole M3")
@@
 	(footprint "MountingHole:MountingHole_3.2mm_M3"
 		(layer "F.Cu")
-		(at 93 143.25)
+		(at 93.3 142.9)
 		(descr "Mounting Hole 3.2mm, M3, no annular, generated by kicad-footprint-generator mountinghole.py")
 		(tags "mountinghole M3")
@@
 	(footprint "MountingHole:MountingHole_3.2mm_M3"
 		(layer "F.Cu")
-		(at 93 52.75)
+		(at 93.3 52.9)
 		(descr "Mounting Hole 3.2mm, M3, no annular, generated by kicad-footprint-generator mountinghole.py")
 		(tags "mountinghole M3")

Commit message: thing thing thing
Parts:
- removed the C10 at (106.6, 124.2)
- removed the J2 at (167.9, 71.6)
- removed the U8 at (104.5, 125.0)
- removed the U9 at (109.3, 125.0)
- added C20: 0.1uF, Capacitor_SMD:C_0402_1005Metric, F.Cu at (107.0, 105.5)
- added SW2: SW_SPST, Button_Switch_SMD:SW_SPDT_Shouhan_MSK12C02, F.Cu at (170.0, 77.0)
- added TP1: SYNC_OUT, TestPoint:TestPoint_Pad_D1.0mm, F.Cu at (165.0, 73.9)
- added U10: TPD4EUSB30, Package_SON:USON-10_2.5x1.0mm_P0.5mm, F.Cu at (103.8, 105.0)
- added U11: TPD4EUSB30, Package_SON:USON-10_2.5x1.0mm_P0.5mm, F.Cu at (111.3, 105.0)
- TP2: renamed from TP1; value TestPoint -> LED0
- moved H4 22.4 mm to (173.3, 122.9)
- moved U8 20.1 mm to (127.9, 116.7)
- moved U6 20.1 mm to (124.6, 104.9)
- moved U7 20.1 mm to (132.1, 104.9)
- moved U12 20.1 mm to (107.4, 116.7)
- moved C10 20.1 mm to (109.1, 98.8)
- moved C12 20.1 mm to (106.4, 92.6)
- moved C13 20.1 mm to (110.4, 97.1)
- moved C14 20.1 mm to (97.0, 98.1)
- moved C18 20.1 mm to (102.3, 98.6)
- moved C19 20.1 mm to (104.5, 93.6)
- moved R4 20.1 mm to (107.4, 91.1)
- moved R5 20.1 mm to (103.2, 98.2)
- moved R6 20.1 mm to (109.7, 91.0)
- moved R7 20.1 mm to (109.7, 90.1)
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- renumbered C12 to C10, C13 to C12, C19 to C13, C17 to C14, C14 to C15, C20 to C16, C15 to C17, C16 to C19, C8 to C3, C5 to C4, C6 to C5, C7 to C6, C4 to C7, C3 to C8, J8 to J2, J6 to J3, R7 to R4, R4 to R5, R5 to R6, R6 to R7, U11 to U1, U7 to U12, U1 to U3, U12 to U4, U10 to U5, U4 to U6, U5 to U7, U3 to U8, U6 to U9
Connections:
- C11 pad 1: /CM5_PCIe/+3.3v -> /+3.3v
- C13 pad 1: /CM5_PCIe/+3.3v -> /+3.3v
- C16 pad 1: /CM5_PCIe/+3.3v -> /+3.3v
- Module1 pad 101: /CM5_GPIO/USB-OTG -> /CM5_HighSpeed/USB_OTG_ID
- Module1 pad 99: /CM5_GPIO/PMIC_ENABLE -> unconnected-(Module1A-PMIC_ENABLE-Pad99)
- R4 pad 2: /CM5_PCIe/+3.3v -> /+3.3v
- R6 pad 1: /CM5_PCIe/+3.3v -> /+3.3v
- U12 pad 15: /CM5_PCIe/+3.3v -> /+3.3v
- U12 pad 17: /CM5_PCIe/+3.3v -> /+3.3v
- U6 pad 10: unconnected-(U4-NC-Pad10) -> /CM5_GPIO/TRD0+
- U6 pad 6: unconnected-(U4-NC-Pad6) -> /CM5_GPIO/TRD1-
- U6 pad 7: unconnected-(U4-NC-Pad7) -> /CM5_GPIO/TRD1+
- U6 pad 9: unconnected-(U4-NC-Pad9) -> /CM5_GPIO/TRD0-
- U7 pad 10: unconnected-(U5-NC-Pad10) (its old number) -> /CM5_GPIO/TRD2+
- U7 pad 6: unconnected-(U5-NC-Pad6) (its old number) -> /CM5_GPIO/TRD3-
- U7 pad 7: unconnected-(U5-NC-Pad7) (its old number) -> /CM5_GPIO/TRD3+
- U7 pad 9: unconnected-(U5-NC-Pad9) (its old number) -> /CM5_GPIO/TRD2-
- U9 pad 11: /CM5_PCIe/+3.3v -> /+3.3v
- U9 pad 23: /CM5_PCIe/+3.3v -> /+3.3v
- U9 pad 32: /CM5_PCIe/+3.3v -> /+3.3v
Routing:
- net /CM5_GPIO/USB-OTG: track 51.6 -> 0.00 mm, vias 2 -> 0
- net /CM5_GPIO/PMIC_ENABLE: track 28.6 -> 0.00 mm
- net /CM5_GPIO/EEPROM_nWP: track 25.8 -> 0.00 mm, vias 2 -> 0
- net /CM5_HighSpeed/PCIe_TX-: track 43.7 -> 23.7 mm
- net /CM5_HighSpeed/PCIe_CLK-: track 39.2 -> 19.2 mm
- net /CM5_HighSpeed/PCIe_nCLKREQ: track 39.2 -> 19.2 mm
- net /CM5_HighSpeed/PCIe_TX+: track 43.7 -> 23.7 mm
- net /CM5_HighSpeed/PCIe_RX-: track 40.4 -> 20.4 mm
- net /CM5_HighSpeed/PCIe_RX+: track 39.8 -> 19.7 mm
- net /CM5_HighSpeed/PCIe_CLK+: track 39.4 -> 19.4 mm
- net /CM5_HighSpeed/PCIe_nRST: track 43.3 -> 23.4 mm
- net /CC1: track 81.9 -> 62.0 mm
- net /USB2_D-: track 73.3 -> 53.7 mm
- net /USB2_D+: track 75.0 -> 55.4 mm
- net /CC2: track 80.5 -> 61.4 mm
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- removed copper zone on In2.Cu, net /CM5_PCIe/+3.3v
Other:
- board size 100 x 100 mm -> 90 x 80 mm

Commit message: pcb for now
Parts:
- removed SW1: SW_Push, Button_Switch_THT:SW_PUSH_6mm
- added J4: Conn_01x02, Connector_PinHeader_2.54mm:PinHeader_1x02_P2.54mm_Vertical, F.Cu at (100.0, 64.2)
- BT1: footprint Battery:BatteryHolder_Keystone_1060_1x2032 -> Battery:BatteryHolder_Keystone_3034_1x20mm
- C20, C5, C6, C9: footprint Capacitor_SMD:C_0402_1005Metric -> Capacitor_SMD:C_0603_1608Metric
- D1, D2: footprint LED_SMD:LED_0402_1005Metric -> LED_SMD:LED_0603_1608Metric
- R1, R2, R3: footprint Resistor_SMD:R_0402_1005Metric -> Resistor_SMD:R_0603_1608Metric
- moved J1 87.0 mm to (102.7, 51.8), turned to 180 degrees
- moved C1 79.7 mm to (100.3, 58.4), turned to -90 degrees
- moved C2 73.6 mm to (105.2, 58.3), turned to -90 degrees
- moved BT1 73.4 mm to (99.2, 80.0)
- moved U1 73.1 mm to (103.2, 60.2), turned to -90 degrees
- moved J2 58.0 mm to (142.8, 111.7), turned to 0 degrees
- moved C4 57.1 mm to (160.5, 107.0)
- moved U2 51.6 mm to (150.7, 105.1)
- moved C3 51.1 mm to (147.7, 104.2), turned to 180 degrees
- moved C6 51.0 mm to (150.1, 109.1), turned to 180 degrees
- moved C5 50.6 mm to (150.1, 107.6), turned to 180 degrees
- moved R1 49.6 mm to (153.5, 106.9), turned to -90 degrees
- moved U5 46.8 mm to (141.5, 106.9), turned to 0 degrees
- moved SW2 14.6 mm to (163.7, 90.2)
- moved D1 10.5 mm to (166.2, 57.3)
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Connections:
- U10 pad 10: /CM5_PCIe/TRD0+ -> unconnected-(U10-NC-Pad10)
- U10 pad 6: /CM5_PCIe/TRD1- -> unconnected-(U10-NC-Pad6)
- U10 pad 7: /CM5_PCIe/TRD1+ -> unconnected-(U10-NC-Pad7)
- U10 pad 9: /CM5_PCIe/TRD0- -> unconnected-(U10-NC-Pad9)
- U11 pad 10: /CM5_PCIe/TRD2+ -> unconnected-(U11-NC-Pad10)
- U11 pad 6: /CM5_PCIe/TRD3- -> unconnected-(U11-NC-Pad6)
- U11 pad 7: /CM5_PCIe/TRD3+ -> unconnected-(U11-NC-Pad7)
- U11 pad 9: /CM5_PCIe/TRD2- -> unconnected-(U11-NC-Pad9)
- U6 pad 10: /CM5_GPIO/TRD0+ -> unconnected-(U6-NC-Pad10)
- U6 pad 6: /CM5_GPIO/TRD1- -> unconnected-(U6-NC-Pad6)
- U6 pad 7: /CM5_GPIO/TRD1+ -> unconnected-(U6-NC-Pad7)
- U6 pad 9: /CM5_GPIO/TRD0- -> unconnected-(U6-NC-Pad9)
- U7 pad 10: /CM5_GPIO/TRD2+ -> unconnected-(U7-NC-Pad10)
- U7 pad 6: /CM5_GPIO/TRD3- -> unconnected-(U7-NC-Pad6)
- U7 pad 7: /CM5_GPIO/TRD3+ -> unconnected-(U7-NC-Pad7)
- U7 pad 9: /CM5_GPIO/TRD2- -> unconnected-(U7-NC-Pad9)
Routing:
- net /CM5_GPIO/VBAT: track 40.0 -> 93.4 mm, vias 0 -> 2
- net /CM5_GPIO/PWR_BUT: track 19.5 -> 57.1 mm, vias 0 -> 1
- net /CM5_HighSpeed/USB3-2-D-: track 23.5 -> 59.5 mm, vias 0 -> 2
- net /CM5_HighSpeed/USB3-2-D+: track 23.5 -> 59.5 mm, vias 0 -> 2
- net /CM5_HighSpeed/USB3-1-D+: track 22.9 -> 56.5 mm
- net /CM5_HighSpeed/USB3-1-D-: track 22.9 -> 56.5 mm
- net GND: track 186.4 -> 159.2 mm, vias 120 -> 124
- net /CM5_HighSpeed/VBUS_EN: track 19.0 -> 39.2 mm, vias 2 -> 0
- net /CM5_GPIO/ETH_LEDY: track 78.6 -> 63.5 mm
- net /CM5_GPIO/ETH_LEDG: track 68.6 -> 55.6 mm
- net /USB2_D+: track 55.4 -> 45.7 mm, vias 0 -> 2
- net /CM5_GPIO/FAN_PWM: track 19.6 -> 10.3 mm
- net /USB2_D-: track 53.7 -> 45.0 mm, vias 0 -> 2
- net /CM5_GPIO/SYNC_OUT: track 23.6 -> 15.0 mm
- net /+3.3v: track 42.6 -> 34.8 mm, vias 6 -> 8
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Other:
- board size 90 x 80 mm -> 80 x 80 mm
- board text removed: "ACT"
- board text removed: "PWR"

Commit message: layout changes
Parts:
- C1, C2, C3: footprint Capacitor_SMD:C_0402_1005Metric -> Capacitor_SMD:C_0603_1608Metric
- R4, R6, R7: footprint Resistor_SMD:R_0402_1005Metric -> Resistor_SMD:R_0603_1608Metric
- moved D1 55.1 mm to (111.6, 49.0), turned to 0 degrees
- moved D2 52.8 mm to (114.6, 49.0), turned to 180 degrees
- moved R2 52.5 mm to (111.7, 51.3), turned to -90 degrees
- moved R3 50.1 mm to (114.3, 51.3), turned to -90 degrees
- moved U2 3.00 mm to (153.7, 105.6)
- moved R4 2.49 mm to (107.7, 88.6), turned to 90 degrees
- moved R6 2.48 mm to (109.2, 88.6), turned to -90 degrees
- moved C3 2.48 mm to (150.1, 104.6)
- moved R7 1.77 mm to (110.7, 88.6), turned to 90 degrees
- moved R1 1.55 mm to (154.2, 108.3), turned to 180 degrees
- moved C2 0.30 mm to (105.2, 58.6)
- moved C1 0.20 mm to (100.3, 58.6)
- moved C5 0.06 mm to (150.1, 107.5)
- moved C6 0.06 mm to (150.1, 109.0)
Connections:
- D1 pad 2: /+3.3v -> /VBUS
- D2 pad 2: /+3.3v -> /VBUS
Routing:
- net /CM5_GPIO/LED_nACT: track 21.8 -> 63.5 mm, vias 2 -> 0
- net /CM5_GPIO/LED_nPWR: track 10.3 -> 50.4 mm
- net /+3.3v: track 34.8 -> 19.8 mm, vias 8 -> 7
- net GND: track 159.2 -> 146.2 mm, vias 124 -> 136
- net /VBUS: track 18.0 -> 21.5 mm, vias 6 -> 7
- net Net-(U9-ISOLATEB): track 5.11 -> 7.12 mm
- net Net-(U9-LANWAKEB): track 2.84 -> 4.81 mm
- net Net-(U2-ILIM): track 2.10 -> 3.71 mm
- net /CM5_HighSpeed/VBUS: track 36.0 -> 34.7 mm
- net /CM5_HighSpeed/VBUS_EN: track 39.2 -> 40.2 mm
- net /CM5_GPIO/FAN_TACHO: track 24.0 -> 23.3 mm
Other:
- board text added: "cm5-router rev 1.0 https://github.com/0x62b/travel-router"

Commit message: stitching via
Routing:
- net GND: vias 136 -> 163
Changed lines of the file:
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@@
+	)
+	(via
+		(at 128.3 124.9)
+		(size 0.6)
+		(drill 0.3)
+		(layers "F.Cu" "B.Cu")
+		(free yes)
+		(net "GND")
 	)
 	(via
@@
 	)
 	(via
+		(at 127.1 82.5)
+		(size 0.6)
+		(drill 0.3)
+		(layers "F.Cu" "B.Cu")
+		(free yes)
+		(net "GND")
+	)
+	(via
 		(at 136.925 69.925)
 		(size 0.6)
@@
 	)
 	(via
+		(at 93.9 117.6)
+		(size 0.6)
+		(drill 0.3)
+		(layers "F.Cu" "B.Cu")
+		(free yes)
+		(net "GND")
+	)
+	(via
 		(at 139.95 69.9)
 		(size 0.6)
@@
 	(via
 		(at 137.05 95.575)
+		(size 0.6)
+		(drill 0.3)
+		(layers "F.Cu" "B.Cu")
+		(free yes)
+		(net "GND")
+	)
+	(via
+		(at 131 70.1)
 		(size 0.6)
 		(drill 0.3)
@@
 	)
 	(via
+		(at 131.1 49)
+		(size 0.6)
+		(drill 0.3)
+		(layers "F.Cu" "B.Cu")
+		(free yes)
+		(net "GND")
+	)
+	(via
 		(at 152.5 63.5)
 		(size 0.6)
@@
 	)
 	(via
+		(at 148 66.6)
+		(size 0.6)
+		(drill 0.3)
+		(layers "F.Cu" "B.Cu")
+		(free yes)
+		(net "GND")
+	)
+	(via
+		(at 92.8 96.2)
+		(size 0.6)
+		(drill 0.3)
+		(layers "F.Cu" "B.Cu")
+		(free yes)
+		(net "GND")
+	)
+	(via
 		(at 162.3 76.2)
 		(size 0.6)
@@
 	)
 	(via
+		(at 155.9 56.4)
+		(size 0.6)
+		(drill 0.3)
+		(layers "F.Cu" "B.Cu")
+		(free yes)
+		(net "GND")
+	)
+	(via
 		(at 139.275 77.325)
 		(size 0.6)
@@
 		(drill 0.3)
 		(layers "F.Cu" "B.Cu")
+		(net "GND")
+	)
+	(via
+		(at 95.5 107.2)
+		(size 0.6)
+		(drill 0.3)
+		(layers "F.Cu" "B.Cu")
+		(free yes)
 		(net "GND")
 	)
@@
 	)
 	(via
+		(at 116 94.5)
+		(size 0.6)
+		(drill 0.3)
+		(layers "F.Cu" "B.Cu")
+		(free yes)
+		(net "GND")
+	)
+	(via
 		(at 140.175 73.8)
 		(size 0.6)
@@
 		(drill 0.3)
 		(layers "F.Cu" "B.Cu")
+		(net "GND")
+	)
+	(via
+		(at 160.1 118.4)
+		(size 0.6)
+		(drill 0.3)
+		(layers "F.Cu" "B.Cu")
+		(free yes)
 		(net "GND")
 	)
@@
 	)
 	(via
+		(at 135.2 57.8)
+		(size 0.6)
+		(drill 0.3)
+		(layers "F.Cu" "B.Cu")
+		(free yes)
+		(net "GND")
+	)
+	(via
 		(at 136.525 77.65)
+		(size 0.6)
+		(drill 0.3)
+		(layers "F.Cu" "B.Cu")
+		(free yes)
+		(net "GND")
+	)
+	(via
+		(at 145.9 73.9)
 		(size 0.6)
 		(drill 0.3)
@@
 	)
 	(via
+		(at 143.3 86.8)
+		(size 0.6)
+		(drill 0.3)
+		(layers "F.Cu" "B.Cu")
+		(free yes)
+		(net "GND")
+	)
+	(via
 		(at 136.95 96.3)
+		(size 0.6)
+		(drill 0.3)
+		(layers "F.Cu" "B.Cu")
+		(free yes)
+		(net "GND")
+	)
+	(via
+		(at 92.8 59.4)
+		(size 0.6)
+		(drill 0.3)
+		(layers "F.Cu" "B.Cu")
+		(free yes)
+		(net "GND")
+	)
+	(via
+		(at 129 52.9)
 		(size 0.6)
 		(drill 0.3)
@@
 	)
 	(via
+		(at 142.964447 51.125103)
+		(size 0.6)
+		(drill 0.3)
+		(layers "F.Cu" "B.Cu")
+		(free yes)
+		(net "GND")
+	)
+	(via
 		(at 132.105 103.78)
 		(size 0.4)
@@
 	)
 	(via
+		(at 146.5 59.4)
+		(size 0.6)
+		(drill 0.3)
+		(layers "F.Cu" "B.Cu")
+		(free yes)
+		(net "GND")
+	)
+	(via
 		(at 139.125 76.5)
 		(size 0.6)
@@
 	)
 	(via
+		(at 165.1 99.8)
+		(size 0.6)
+		(drill 0.3)
+		(layers "F.Cu" "B.Cu")
+		(free yes)
+		(net "GND")
+	)
+	(via
 		(at 136.5 96.825)
 		(size 0.6)
@@
 	)
 	(via
+		(at 132.7 91.8)
+		(size 0.6)
+		(drill 0.3)
+		(layers "F.Cu" "B.Cu")
+		(free yes)
+		(net "GND")
+	)
+	(via
 		(at 139.35 72.775)
 		(size 0.6)
@@
 	)
 	(via
+		(at 126.2 91.8)
+		(size 0.6)
+		(drill 0.3)
+		(layers "F.Cu" "B.Cu")
+		(free yes)
+		(net "GND")
+	)
+	(via
+		(at 127.1 113.6)
+		(size 0.6)
+		(drill 0.3)
+		(layers "F.Cu" "B.Cu")
+		(free yes)
+		(net "GND")
+	)
+	(via
 		(at 124.2 77.1)
 		(size 0.6)
@@
 		(drill 0.3)
 		(layers "F.Cu" "B.Cu")
+		(net "GND")
+	)
+	(via
+		(at 161.1 62.5)
+		(size 0.6)
+		(drill 0.3)
+		(layers "F.Cu" "B.Cu")
+		(free yes)
 		(net "GND")
 	)
@@
 	)
 	(via
+		(at 147 121)
+		(size 0.6)
+		(drill 0.3)
+		(layers "F.Cu" "B.Cu")
+		(free yes)
+		(net "GND")
+	)
+	(via
 		(at 136.5 76.9)
 		(size 0.6)
@@
 	)
 	(via
+		(at 164.6 57.5)
+		(size 0.6)
+		(drill 0.3)
+		(layers "F.Cu" "B.Cu")
+		(free yes)
+		(net "GND")
+	)
+	(via
+		(at 165.6 112.5)
+		(size 0.6)
+		(drill 0.3)
+		(layers "F.Cu" "B.Cu")
+		(free yes)
+		(net "GND")
+	)
+	(via
 		(at 151.8 78.9)
 		(size 0.6)
@@
 		(size 0.6)
 		(drill 0.3)
+		(layers "F.Cu" "B.Cu")
+		(free yes)
+		(net "GND")
+	)
+	(via
+		(at 146.8 105.6)
+		(size 0.6)
+		(drill 0.3)

Commit message: (probably) final pcb
Parts:
- added G***: LOGO, LOGO, B.Cu at (128.3, 87.9)
Routing:
- net GND: track 146.2 -> 130.3 mm, vias 163 -> 152
- net /CM5_GPIO/TRD3-: track 49.3 -> 44.4 mm, vias 2 -> 0
- net /CM5_HighSpeed/PCIe_nRST: track 23.4 -> 27.8 mm
- net /CM5_PCIe/TRD1+: track 10.9 -> 14.8 mm
- net /CM5_GPIO/TRD1+: track 44.3 -> 47.8 mm, vias 2 -> 0
- net /CM5_PCIe/TRD3+: track 11.8 -> 15.3 mm
- net /CM5_HighSpeed/USB3-2-D-: track 59.5 -> 62.4 mm
- net /CM5_HighSpeed/USB3-1-D+: track 56.5 -> 59.0 mm
- net /CM5_HighSpeed/USB3-1-D-: track 56.5 -> 58.9 mm
- net /CM5_HighSpeed/USB3-2-D+: track 59.5 -> 61.8 mm
- net /CM5_GPIO/TRD0-: track 49.5 -> 47.3 mm, vias 2 -> 0
- net /CM5_GPIO/TRD2-: track 46.4 -> 44.3 mm, vias 2 -> 0
- net /CM5_PCIe/TRD2+: track 11.9 -> 13.5 mm
- net /CM5_PCIe/TRD0+: track 12.1 -> 13.6 mm
- net /CM5_GPIO/TRD0+: track 48.5 -> 47.2 mm, vias 2 -> 0
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
Commit message: update
Routing:
- net /CM5_GPIO/FAN_TACHO: track 23.3 -> 22.6 mm
