File: pcb/cm5_highspeed.kicad_sch (KiCad schematic)
At the start: 12 parts, among them J5 HDMI_A, J8 USB_A_Stacked, U1 RT9742SNGV, U2 AP2553W6

Commit message: thing
Parts:
- removed J5: HDMI_A, Connector_Video:HDMI_A_Molex_208658-1001_Horizontal, symbol Connector:HDMI_A
- added U10: TPD4EUSB30, Package_SON:USON-10_2.5x1.0mm_P0.5mm, symbol Power_Protection:TPD4EUSB30
- added U12: 476591100, easyeda2kicad:HDMI-SMD_19P-P0.50_0476591102, symbol easyeda2kicad:476591100
Connections:
- net GND: now also U12.1 (TMDS_Data2_Shield), U12.10 (TMDS_Clock_Shield), U12.13 (DDC/CEC_Ground), U12.21 (EH), U12.22 (EH), U12.23 (EH), U12.4 (TMDS_Data1_Shield), U12.7 (TMDS_Data0_Shield)
- net HDMI0_CEC: now also U12.14 (CEC)
- net HDMI0_CLK+: now also U12.11 (TMDS_Clock+)
- net HDMI0_CLK-: now also U12.12 (TMDS_Clock-)
- net HDMI0_HOTPLUG: now also U12.19 (HotPlugDetect/HEAC-)
- net HDMI0_SCL: now also U12.15 (SCL)
- net HDMI0_SDA: now also U12.16 (SDA)
- net HDMI0_TX0+: now also U12.8 (TMDS_Data0+)
- net HDMI0_TX0-: now also U12.9 (TMDS_Data0-)
- net HDMI0_TX1+: now also U12.5 (TMDS_Data1+)
- net HDMI0_TX1-: now also U12.6 (TMDS_Data1-)
- net HDMI0_TX2+: now also U12.2 (TMDS_Data2+)
- net HDMI0_TX2-: now also U12.3 (TMDS_Data2-)
- net HDMI_5V: now also U12.18 (+5VPower)
- net USB3-1-D+: now also J8.3 (D1+), U10.4 (D2+); no longer J8.7 (D2+)
- net USB3-1-D-: now also J8.2 (D1-), U10.5 (D2-); no longer J8.6 (D2-)
- net USB3-2-D+: now also J8.7 (D2+), U10.1 (D1+); no longer J8.2 (D1-)
- net USB3-2-D-: now also J8.6 (D2-), U10.2 (D1-); no longer J8.3 (D1+)
- new net: U10.3 (GND), U10.8 (GND)
Other:
- moved on the sheet: J8

Commit message: thing thing thing
Parts:
- renumbered C8 to C3, C5 to C4, C6 to C5, C7 to C6, C4 to C7, C3 to C8, J8 to J2, U1 to U3, U12 to U4, U10 to U5
Changed lines of the file:
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@@
 		(dnp no)
 		(fields_autoplaced yes)
-		(property "Reference" "#PWR02"
+		(property "Reference" "#PWR07"
 			(at 96.52 194.31 0)
 			(hide yes)
@@
 			(project "travel-router"
 				(path "/10ff01a9-f304-4749-ad89-df55c3f3b44a/513e9443-5f2e-4ddd-b8ed-a2c4fe5dd9e2"
-					(reference "#PWR02")
+					(reference "#PWR07")
 					(unit 1)
 				)
@@
 		(dnp no)
 		(fields_autoplaced yes)
-		(property "Reference" "#PWR010"
+		(property "Reference" "#PWR014"
 			(at 220.98 96.52 0)
 			(hide yes)
@@
 			(project "travel-router"
 				(path "/10ff01a9-f304-4749-ad89-df55c3f3b44a/513e9443-5f2e-4ddd-b8ed-a2c4fe5dd9e2"
-					(reference "#PWR010")
+					(reference "#PWR014")
 					(unit 1)
 				)
@@
 		(dnp no)
 		(fields_autoplaced yes)
-		(property "Reference" "U10"
+		(property "Reference" "U5"
 			(at 252.73 120.65 0)
 			(show_name no)
@@
 			(project "travel-router"
 				(path "/10ff01a9-f304-4749-ad89-df55c3f3b44a/513e9443-5f2e-4ddd-b8ed-a2c4fe5dd9e2"
-					(reference "U10")
+					(reference "U5")
 					(unit 1)
 				)
@@
 		(dnp no)
 		(fields_autoplaced yes)
-		(property "Reference" "#PWR013"
+		(property "Reference" "#PWR09"
 			(at 129.54 190.5 0)
 			(hide yes)
@@
 			(project "travel-router"
 				(path "/10ff01a9-f304-4749-ad89-df55c3f3b44a/513e9443-5f2e-4ddd-b8ed-a2c4fe5dd9e2"
-					(reference "#PWR013")
+					(reference "#PWR09")
 					(unit 1)
 				)
@@
 		(dnp no)
 		(fields_autoplaced yes)
-		(property "Reference" "#PWR07"
+		(property "Reference" "#PWR016"
 			(at 267.97 62.23 0)
 			(hide yes)
@@
 			(project "travel-router"
 				(path "/10ff01a9-f304-4749-ad89-df55c3f3b44a/513e9443-5f2e-4ddd-b8ed-a2c4fe5dd9e2"
-					(reference "#PWR07")
+					(reference "#PWR016")
 					(unit 1)
 				)
@@
 		(dnp no)
 		(fields_autoplaced yes)
-		(property "Reference" "U12"
+		(property "Reference" "U4"
 			(at 231.14 19.05 0)
 			(show_name no)
@@
 			(project "travel-router"
 				(path "/10ff01a9-f304-4749-ad89-df55c3f3b44a/513e9443-5f2e-4ddd-b8ed-a2c4fe5dd9e2"
-					(reference "U12")
+					(reference "U4")
 					(unit 1)
 				)
@@
 		(dnp no)
 		(fields_autoplaced yes)
-		(property "Reference" "#PWR08"
+		(property "Reference" "#PWR011"
 			(at 194.31 62.23 0)
 			(hide yes)
@@
 			(project "travel-router"
 				(path "/10ff01a9-f304-4749-ad89-df55c3f3b44a/513e9443-5f2e-4ddd-b8ed-a2c4fe5dd9e2"
-					(reference "#PWR08")
+					(reference "#PWR011")
 					(unit 1)
 				)
@@
 		(dnp no)
 		(fields_autoplaced yes)
-		(property "Reference" "#PWR04"
+		(property "Reference" "#PWR08"
 			(at 123.19 161.29 0)
 			(hide yes)
@@
 			(project "travel-router"
 				(path "/10ff01a9-f304-4749-ad89-df55c3f3b44a/513e9443-5f2e-4ddd-b8ed-a2c4fe5dd9e2"
-					(reference "#PWR04")
+					(reference "#PWR08")
 					(unit 1)
 				)
@@
 		(dnp no)
 		(fields_autoplaced yes)
-		(property "Reference" "#PWR035"
+		(property "Reference" "#PWR012"
 			(at 195.58 158.75 0)
 			(hide yes)
@@
 			(project "travel-router"
 				(path "/10ff01a9-f304-4749-ad89-df55c3f3b44a/513e9443-5f2e-4ddd-b8ed-a2c4fe5dd9e2"
-					(reference "#PWR035")
+					(reference "#PWR012")
 					(unit 1)
 				)
@@
 		(dnp no)
 		(fields_autoplaced yes)
-		(property "Reference" "#PWR012"
+		(property "Reference" "#PWR06"
 			(at 76.2 185.42 0)
 			(hide yes)
@@
 			(project "travel-router"
 				(path "/10ff01a9-f304-4749-ad89-df55c3f3b44a/513e9443-5f2e-4ddd-b8ed-a2c4fe5dd9e2"
-					(reference "#PWR012")
+					(reference "#PWR06")
 					(unit 1)
 				)
@@
 		(dnp no)
 		(fields_autoplaced yes)
-		(property "Reference" "J8"
+		(property "Reference" "J2"
 			(at 193.04 118.11 0)
 			(show_name no)
@@
 			(project "travel-router"
 				(path "/10ff01a9-f304-4749-ad89-df55c3f3b44a/513e9443-5f2e-4ddd-b8ed-a2c4fe5dd9e2"
-					(reference "J8")
+					(reference "J2")
 					(unit 1)
 				)
@@
 		(dnp no)
 		(fields_autoplaced yes)
-		(property "Reference" "#PWR027"
+		(property "Reference" "#PWR015"
 			(at 236.22 62.23 0)
 			(hide yes)
@@
 			(project "travel-router"
 				(path "/10ff01a9-f304-4749-ad89-df55c3f3b44a/513e9443-5f2e-4ddd-b8ed-a2c4fe5dd9e2"
-					(reference "#PWR027")
+					(reference "#PWR015")
 					(unit 1)
 				)
@@
 		(dnp no)
 		(fields_autoplaced yes)
-		(property "Reference" "U1"
+		(property "Reference" "U3"
 			(at 207.01 73.66 0)
 			(show_name no)
@@
 			(project "travel-router"
 				(path "/10ff01a9-f304-4749-ad89-df55c3f3b44a/513e9443-5f2e-4ddd-b8ed-a2c4fe5dd9e2"
-					(reference "U1")
+					(reference "U3")
 					(unit 1)
 				)
@@
 		(dnp no)
 		(fields_autoplaced yes)
-		(property "Reference" "#PWR011"
+		(property "Reference" "#PWR010"
 			(at 190.5 96.52 0)
 			(hide yes)
@@
 			(project "travel-router"
 				(path "/10ff01a9-f304-4749-ad89-df55c3f3b44a/513e9443-5f2e-4ddd-b8ed-a2c4fe5dd9e2"
-					(reference "#PWR011")
+					(reference "#PWR010")
 					(unit 1)
 				)
@@
 		(dnp no)
 		(fields_autoplaced yes)
-		(property "Reference" "C5"
+		(property "Reference" "C4"
 			(at 106.68 175.6409 0)
 			(show_name no)
@@
 			(project "travel-router"
 				(path "/10ff01a9-f304-4749-ad89-df55c3f3b44a/513e9443-5f2e-4ddd-b8ed-a2c4fe5dd9e2"
-					(reference "C5")
+					(reference "C4")
 					(unit 1)
 				)
@@
 		(dnp no)
 		(fields_autoplaced yes)
-		(property "Reference" "C8"
+		(property "Reference" "C3"
 			(at 58.42 175.2599 0)
 			(show_name no)
@@
 			(project "travel-router"
 				(path "/10ff01a9-f304-4749-ad89-df55c3f3b44a/513e9443-5f2e-4ddd-b8ed-a2c4fe5dd9e2"
-					(reference "C8")
+					(reference "C3")
 					(unit 1)
 				)
@@
 		(dnp no)
 		(fields_autoplaced yes)
-		(property "Reference" "C7"
+		(property "Reference" "C6"
 			(at 133.35 176.5299 0)
 			(show_name no)
@@
 			(project "travel-router"
 				(path "/10ff01a9-f304-4749-ad89-df55c3f3b44a/513e9443-5f2e-4ddd-b8ed-a2c4fe5dd9e2"
-					(reference "C7")
+					(reference "C6")
 					(unit 1)
 				)
@@
 		(dnp no)
 		(fields_autoplaced yes)
-		(property "Reference" "#PWR014"
+		(property "Reference" "#PWR04"
 			(at 54.61 187.96 0)
 			(hide yes)
@@
 			(project "travel-router"
 				(path "/10ff01a9-f304-4749-ad89-df55c3f3b44a/513e9443-5f2e-4ddd-b8ed-a2c4fe5dd9e2"
-					(reference "#PWR014")
+					(reference "#PWR04")
 					(unit 1)
 				)
@@
 		(dnp no)
 		(fields_autoplaced yes)
-		(property "Reference" "C4"
+		(property "Reference" "C7"
 			(at 194.31 83.8199 0)
 			(show_name no)
@@
 			(project "travel-router"
 				(path "/10ff01a9-f304-4749-ad89-df55c3f3b44a/513e9443-5f2e-4ddd-b8ed-a2c4fe5dd9e2"
-					(reference "C4")
+					(reference "C7")
 					(unit 1)
 				)
@@
 		(dnp no)
 		(fields_autoplaced yes)
-		(property "Reference" "C3"
+		(property "Reference" "C8"
 			(at 224.79 83.8199 0)
 			(show_name no)
@@
 			(project "travel-router"
 				(path "/10ff01a9-f304-4749-ad89-df55c3f3b44a/513e9443-5f2e-4ddd-b8ed-a2c4fe5dd9e2"
-					(reference "C3")
+					(reference "C8")
 					(unit 1)
 				)
@@
 		(dnp no)
 		(fields_autoplaced yes)
-		(property "Reference" "#PWR09"
+		(property "Reference" "#PWR013"
 			(at 207.01 96.52 0)
 			(hide yes)
@@
 			(project "travel-router"
 				(path "/10ff01a9-f304-4749-ad89-df55c3f3b44a/513e9443-5f2e-4ddd-b8ed-a2c4fe5dd9e2"
-					(reference "#PWR09")
+					(reference "#PWR013")
 					(unit 1)
 				)
@@
 		(dnp no)
 		(fields_autoplaced yes)
-		(property "Reference" "C6"
+		(property "Reference" "C5"
 			(at 121.92 176.5299 0)
 			(show_name no)
@@
 			(project "travel-router"
 				(path "/10ff01a9-f304-4749-ad89-df55c3f3b44a/513e9443-5f2e-4ddd-b8ed-a2c4fe5dd9e2"
-					(reference "C6")
+					(reference "C5")
 					(unit 1)
 				)

Commit message: pcb for now
Parts:
- C5, C6: footprint Capacitor_SMD:C_0402_1005Metric -> Capacitor_SMD:C_0603_1608Metric
- R1: footprint Resistor_SMD:R_0402_1005Metric -> Resistor_SMD:R_0603_1608Metric
Changed lines of the file:
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@@
 			)
 		)
-		(property "Footprint" "Capacitor_SMD:C_0402_1005Metric"
+		(property "Footprint" "Capacitor_SMD:C_0603_1608Metric"
 			(at 130.5052 181.61 0)
 			(hide yes)
@@
 			)
 		)
-		(property "Footprint" "Resistor_SMD:R_0402_1005Metric"
+		(property "Footprint" "Resistor_SMD:R_0603_1608Metric"
 			(at 94.742 182.88 90)
 			(hide yes)
@@
 			)
 		)
-		(property "Footprint" "Capacitor_SMD:C_0402_1005Metric"
+		(property "Footprint" "Capacitor_SMD:C_0603_1608Metric"
 			(at 119.0752 181.61 0)
 			(hide yes)

Commit message: layout changes
Parts:
- C3: footprint Capacitor_SMD:C_0402_1005Metric -> Capacitor_SMD:C_0603_1608Metric
Changed lines of the file:
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@@
 			)
 		)
-		(property "Footprint" "Capacitor_SMD:C_0402_1005Metric"
+		(property "Footprint" "Capacitor_SMD:C_0603_1608Metric"
 			(at 55.5752 180.34 0)
 			(hide yes)
